Commit message: feat(SWM25-46): configure ROSOrin robot assets

File: malbut_description/urdf/materials.xacro (robot description, xacro)
@@ -1,27 +1,18 @@
 <?xml version="1.0"?>
-<robot>
-    <material name="black">
-        <color rgba="0.3 0.3 0.3 1.0"/>
-    </material>
-    <material name="blue">
-        <color rgba="0.0 0.0 0.8 1.0"/>
-    </material>
-    <material name="green">
-        <color rgba="0.4 0.9 0.4 1.0"/>
-    </material>
-    <material name="gray">
-        <color rgba="0.7 0.7 0.7 1.0"/>
-    </material>
-    <material name="darkgray">
-        <color rgba="0.3 0.3 0.3 1.0"/>
-    </material>
-    <material name="red">
-        <color rgba="0.8 0.0 0.0 1.0"/>
-    </material>
-    <material name="white">
-        <color rgba="1.0 1.0 1.0 1.0"/>
-    </material>
-    <material name="yellow">
-        <color rgba="0.8 0.8 0.0 1.0"/>
-    </material>
+<robot xmlns:xacro="http://www.ros.org/wiki/xacro">
+  <material name="rosorin_orange">
+    <color rgba="0.95 0.30 0.04 1.0"/>
+  </material>
+  <material name="rosorin_dark">
+    <color rgba="0.08 0.09 0.11 1.0"/>
+  </material>
+  <material name="rosorin_aluminum">
+    <color rgba="0.55 0.58 0.62 1.0"/>
+  </material>
+  <material name="rosorin_sensor">
+    <color rgba="0.12 0.20 0.28 1.0"/>
+  </material>
+  <material name="rosorin_lens">
+    <color rgba="0.05 0.20 0.32 0.85"/>
+  </material>
 </robot>

File: malbut_description/urdf/rosorin.xacro (robot description, xacro)
@@ -1,366 +1,11 @@
-<?xml version="1.0" encoding="utf-8"?>
-<robot name="car" xmlns:xacro="http://ros.org/wiki/xacro" >
-  <xacro:arg name="camera_type" default="$(optenv DEPTH_CAMERA_TYPE aurora)"/>
-  <xacro:property name="camera_type" value="$(arg camera_type)"/>
-  <xacro:include filename="$(find malbut_description)/urdf/materials.xacro"/>
-  <link name="base_footprint"/>
-  <joint name="base_joint" type="fixed">
-    <parent link="base_footprint"/>
-    <child link="base_link"/>
-    <origin xyz="0.0 0.0 0.028" rpy="0 0 0"/>
-  </joint>
-  <link name="imu_link"/>
-  <joint name="imu_joint" type="fixed">
-    <parent link="base_link"/>
-    <child link="imu_link"/>
-    <origin xyz="0.04 -0.015 0.05" rpy="0 0 1.57"/>
-  </joint>
-  <link
-    name="base_link">
-    <inertial>
-      <origin
-        xyz="-0.0073743 0.00027245 0.033869"
-        rpy="0 0 0" />
-      <mass
-        value="0.05536" />
-      <inertia
-        ixx="0.00029526"
-        ixy="-8.622E-07"
-        ixz="3.753E-05"
-        iyy="0.00065872"
-        iyz="-4.6067E-09"
-        izz="0.00086726" />
-    </inertial>
-    <visual>
-      <origin
-        xyz="0 0 0"
-        rpy="0 0 0" />
-      <geometry>
-        <mesh
-          filename="file://$(find malbut_description)/meshes/base_link.stl" />
-      </geometry>
-      <material
-        name="">
-        <color
-          rgba="0.5 0.5 0.5 1" />
-      </material>
-    </visual>
-    <collision>
-      <origin
-        xyz="0 0 0"
-        rpy="0 0 0" />
-      <geometry>
-        <mesh
-          filename="file://$(find malbut_description)/meshes/base_link_collision.stl" />
-      </geometry>
-    </collision>
-  </link>
-  <link
-    name="lidar_frame">
-    <inertial>
-      <origin
-        xyz="8.95497003335615E-05 6.44963541535514E-05 -0.011400348556056"
-        rpy="0 0 0" />
-      <mass
-        value="0.0385600938526619" />
-      <inertia
-        ixx="4.66264138781846E-06"
-        ixy="-1.60730633906311E-07"
-        ixz="2.05163088641334E-09"
-        iyy="4.71595831823178E-06"
-        iyz="1.10063023333176E-08"
-        izz="7.61240253383846E-06" />
-    </inertial>
-    <visual>
-      <origin
-        xyz="0 0 0"
-        rpy="0 0 0" />
-      <geometry>
-        <mesh
-          filename="file://$(find malbut_description)/meshes/lidar_link.stl" />
-      </geometry>
-      <material name="black"/>
-    </visual>
-    <collision>
-      <origin
-        xyz="0 0 0"
-        rpy="0 0 0" />
-      <geometry>
-        <mesh
-          filename="file://$(find malbut_description)/meshes/lidar_link_collision.stl" />
-      </geometry>
-    </collision>
-  </link>
-  <joint
-    name="lidar"
-    type="fixed">
-    <origin
-      xyz="0.011476 7.415E-05 0.13641"
-      rpy="0 0 0" />
-    <parent
-      link="base_link" />
-    <child
-      link="lidar_frame" />
-    <axis
-      xyz="0 0 0" />
-  </joint>
-  <link
-    name="left_front_wheel_link">
-    <inertial>
-      <origin
-        xyz="6.78850066051367E-05 0.0194273902243469 4.2771032181671E-05"
-        rpy="0 0 0" />
-      <mass
-        value="0.0705101646075632" />
-      <inertia
-        ixx="1.05359955410655E-05"
-        ixy="-4.17160486096137E-09"
-        ixz="-3.48250757597355E-08"
-        iyy="1.65950885885739E-05"
-        iyz="4.89765791745149E-09"
-        izz="1.05450583464434E-05" />
-    </inertial>
-    <visual>
-      <origin
-        xyz="0 0 0"
-        rpy="0 0 0" />
-      <geometry>
-        <mesh
-          filename="file://$(find malbut_description)/meshes/left_front_wheel_link.stl" />
-      </geometry>
-      <material name="black"/>
-    </visual>
-    <collision>
-      <origin
-        xyz="0 0 0"
-        rpy="0 0 0" />
-      <geometry>
-        <mesh
-          filename="file://$(find malbut_description)/meshes/left_front_wheel_link_collision.stl" />
-      </geometry>
-    </collision>
-  </link>
-  <joint
-    name="left_front_wheel"
-    type="fixed">
-    <origin
-      xyz="0.09097 0.067865 0.017096"
-      rpy="0 0 0" />
-    <parent
-      link="base_link" />
-    <child
-      link="left_front_wheel_link" />
-    <axis
-      xyz="0 0 0" />
-  </joint>
-  <link
-    name="left_back_wheel_link">
-    <inertial>
-      <origin
-        xyz="-6.79935957126898E-05 0.0194272724865622 4.18919442857144E-05"
-        rpy="0 0 0" />
-      <mass
-        value="0.0705098315712721" />
-      <inertia
-        ixx="1.05363965532436E-05"
-        ixy="4.22186803055192E-09"
-        ixz="3.45056141524137E-08"
-        iyy="1.65964488067E-05"
-        iyz="4.90631628693761E-09"
-        izz="1.05458413899706E-05" />
-    </inertial>
-    <visual>
-      <origin
-        xyz="0 0 0"
-        rpy="0 0 0" />
-      <geometry>
-        <mesh
-          filename="file://$(find malbut_description)/meshes/left_back_wheel_link.stl" />
-      </geometry>
-      <material name="black"/>
-    </visual>
-    <collision>
-      <origin
-        xyz="0 0 0"
-        rpy="0 0 0" />
-      <geometry>
-        <mesh
-          filename="file://$(find malbut_description)/meshes/left_back_wheel_link_collision.stl" />
-      </geometry>
-    </collision>
-  </link>
-  <joint
-    name="left_back_wheel"
-    type="fixed">
-    <origin
-      xyz="-0.080677 0.067865 0.016719"
-      rpy="0 0 0" />
-    <parent
-      link="base_link" />
-    <child
-      link="left_back_wheel_link" />
-    <axis
-      xyz="0 0 0" />
-  </joint>
-  <link
-    name="right_front_wheel_link">
-    <inertial>
-      <origin
-        xyz="6.56410494759008E-05 -0.0194272432930035 4.09111593353481E-05"
-        rpy="0 0 0" />
-      <mass
-        value="0.0705098464929629" />
-      <inertia
-        ixx="1.0536754444795E-05"
-        ixy="4.2338086716559E-09"
-        ixz="-3.43871505647673E-08"
-        iyy="1.6596872052673E-05"
-        iyz="-4.91902435337096E-09"
-        izz="1.05459220480947E-05" />
-    </inertial>
-    <visual>
-      <origin
-        xyz="0 0 0"
-        rpy="0 0 0" />
-      <geometry>
-        <mesh
-          filename="file://$(find malbut_description)/meshes/right_front_wheel_link.stl" />
-      </geometry>
-      <material name="black"/>
-    </visual>
-    <collision>
-      <origin
-        xyz="0 0 0"
-        rpy="0 0 0" />
-      <geometry>
-        <mesh
-          filename="file://$(find malbut_description)/meshes/right_front_wheel_link_collision.stl" />
-      </geometry>
-    </collision>
-  </link>
-  <joint
-    name="right_front_wheel"
-    type="fixed">
-    <origin
-      xyz="0.090972 -0.067717 0.017098"
-      rpy="0 0 0" />
-    <parent
-      link="base_link" />
-    <child
-      link="right_front_wheel_link" />
-    <axis
-      xyz="0 0 0" />
-  </joint>
-  <link
-    name="right_back_wheel_link">
-    <inertial>
-      <origin
-        xyz="-4.8854E-05 -0.017043 1.8927E-05"
-        rpy="0 0 0" />
-      <mass
-        value="0.058672" />
-      <inertia
-        ixx="6.7699E-06"
-        ixy="-1.99E-08"
-        ixz="1.4456E-08"
-        iyy="9.6881E-06"
-        iyz="1.0739E-08"
-        izz="6.7781E-06" />
-    </inertial>
-    <visual>
-      <origin
-        xyz="0 0 0"
-        rpy="0 0 0" />
-      <geometry>
-        <mesh
-          filename="file://$(find malbut_description)/meshes/right_back_wheel_link.stl" />
-      </geometry>
-      <material name="black"/>
-    </visual>
-    <collision>
-      <origin
-        xyz="0 0 0"
-        rpy="0 0 0" />
-      <geometry>
-        <mesh
-          filename="file://$(find malbut_description)/meshes/right_back_wheel_link_collision.stl" />
-      </geometry>
-    </collision>
-  </link>
-  <joint
-    name="right_back_wheel"
-    type="fixed">
-    <origin
-      xyz="-0.080677 -0.067717 0.016719"
-      rpy="0 0 0" />
-    <parent
-      link="base_link" />
-    <child
-      link="right_back_wheel_link" />
-    <axis
-      xyz="0 0 0" />
-  </joint>
-  <link
-    name="mic_link">
-    <inertial>
-      <origin
-        xyz="-7.65493159082808E-07 -0.0249662719365599 0.0134328993494675"
-        rpy="0 0 0" />
-      <mass
-        value="0.0210934941268813" />
-      <inertia
-        ixx="1.36191114404946E-05"
-        ixy="-4.3417522172067E-10"
-        ixz="-1.27861440031619E-10"
-        iyy="3.01739703567571E-05"
-        iyz="4.99987016844085E-11"
-        izz="4.19372593423754E-05" />
-    </inertial>
-    <visual>
-      <origin
-        xyz="0 0 0"
-        rpy="0 0 0" />
-      <geometry>
-        <mesh
-          filename="file://$(find malbut_description)/meshes/mic_link.stl" />
-      </geometry>
-      <material name="black"/>
-    </visual>
-    <collision>
-      <origin
-        xyz="0 0 0"
-        rpy="0 0 0" />
-      <geometry>
-        <mesh
-          filename="file://$(find malbut_description)/meshes/mic_link_collision.stl" />
-      </geometry>
-    </collision>
-  </link>
-  <joint
-    name="mic"
-    type="fixed">
-    <origin
-      xyz="-0.068965 0.025075 0.10955"
-      rpy="0 0 0" />
-    <parent
-      link="base_link" />
-    <child
-      link="mic_link" />
-    <axis
-      xyz="0 0 0" />
-  </joint>
-  <link name="lidar_sim_frame" />
-  <joint
-    name="lidar_sim_frame_joint"
-    type="fixed">
-    <origin xyz="0 0 0" rpy="0 0 0" />
-    <parent link="lidar_frame" />
-    <child link="lidar_sim_frame" />
-  </joint>
-  <xacro:if value="${camera_type == 'AsCamera' or camera_type == 'aurora'}">
-    <xacro:include filename="$(find malbut_description)/urdf/ascamera.xacro"/>
-  </xacro:if>
-  <xacro:if value="${camera_type == 'Dabai'}">
-    <xacro:include filename="$(find malbut_description)/urdf/dabai.xacro"/>
-  </xacro:if>
+<?xml version="1.0"?>
+<robot
+  name="malbut_rosorin_ultimate_orin_nx_super"
+  xmlns:xacro="http://www.ros.org/wiki/xacro">
+  <!--
+    Stable public entry point retained for existing launch files.
+    Tunable values are declared by rosorin_model.xacro and mirrored in config/.
+  -->
+  <xacro:include filename="$(find malbut_description)/urdf/rosorin_model.xacro"/>
+  <xacro:rosorin_model/>
 </robot>

File: malbut_gazebo/urdf/robot.gazebo.xacro (robot description, xacro)
@@ -1,58 +1,10 @@
-<?xml version="1.0" encoding="utf-8"?>
-<robot name="robot" xmlns:xacro="http://ros.org/wiki/xacro">
-    <xacro:arg name="sim_ign" default="true"/>
-    <!-- robot_description -->
-    <xacro:include filename="$(find malbut_description)/urdf/rosorin.xacro"/>
-    <xacro:if value="$(arg sim_ign)">
-        <xacro:include filename="$(find malbut_gazebo)/urdf/wheel.xacro"/>
-    </xacro:if>
-    <!-- lidar -->
-    <xacro:include filename="$(find malbut_gazebo)/urdf/lidar.gazebo.xacro"/>
-    <!-- camera -->
-    <xacro:include filename="$(find malbut_gazebo)/urdf/camera.gazebo.xacro"/>
-    <xacro:if value="${camera_type == 'AsCamera' or camera_type == 'aurora'}">
-        <xacro:gazebo_camera reference="camera_link0"/>
-    </xacro:if>
-    <xacro:if value="${camera_type == 'Dabai'}">
-        <xacro:gazebo_camera reference="depth_cam_link"/>
-    </xacro:if>
-    <!-- imu -->
-    <xacro:include filename="$(find malbut_gazebo)/urdf/imu.gazebo.xacro"/>
-    <gazebo>
-        <!-- Joint state publisher -->
-        <plugin filename="libignition-gazebo-joint-state-publisher-system.so" name="ignition::gazebo::systems::JointStatePublisher">
-            <topic>joint_states</topic>
-        </plugin>
-        <!-- sensor-liar -->
-        <plugin filename="ignition-gazebo-sensors-system" name="ignition::gazebo::systems::Sensors">
-            <render_engine>ogre2</render_engine>
-        </plugin>
-        <!-- imu -->
-        <plugin filename="ignition-gazebo-imu-system" name="ignition::gazebo::systems::Imu"></plugin>
-        <!-- odom -->
-        <plugin
-            filename="ignition-gazebo-odometry-publisher-system"
-            name="ignition::gazebo::systems::OdometryPublisher">
-            <odom_publish_frequency>50</odom_publish_frequency>
-            <odom_topic>/odom</odom_topic>
-            <odom_frame>odom</odom_frame>
-            <robot_base_frame>base_footprint</robot_base_frame>
-            <tf_topic>/odom/tf</tf_topic>
-        </plugin>
-        <xacro:if value="$(arg sim_ign)">
-            <plugin filename="ignition-gazebo-mecanum-drive-system" name="ignition::gazebo::systems::MecanumDrive">
-                <front_left_joint>front_left_joint</front_left_joint>
-                <front_right_joint>front_right_joint</front_right_joint>
-                <back_left_joint>rear_left_joint</back_left_joint>
-                <back_right_joint>rear_right_joint</back_right_joint>
-                <wheel_separation>0.34</wheel_separation>
-                <wheelbase>0.3</wheelbase>
-                <wheel_radius>0.05</wheel_radius>
-                <topic>/controller/cmd_vel</topic>
-                <odom_topic>/odom</odom_topic>
-                <frame_id>odom</frame_id>
-                <child_frame_id>base_link</child_frame_id>
-            </plugin>
-        </xacro:if>
-    </gazebo>
+<?xml version="1.0"?>
+<robot
+  name="malbut_rosorin_ultimate_orin_nx_super"
+  xmlns:xacro="http://www.ros.org/wiki/xacro"
+  xmlns:ignition="http://ignitionrobotics.org/schema">
+  <xacro:include filename="$(find malbut_description)/urdf/rosorin_model.xacro"/>
+  <xacro:include filename="$(find malbut_gazebo)/urdf/gazebo_plugins.xacro"/>
+  <xacro:rosorin_model/>
+  <xacro:rosorin_gazebo/>
 </robot>
