Commit message: fix(SWM25-58): separate RGB and depth camera clip ranges

File: malbut_description/urdf/rosorin_model.xacro (robot description, xacro)
@@ -45,5 +45,7 @@
   <xacro:arg name="camera_hfov" default="1.291543646"/>
   <xacro:arg name="camera_near" default="0.15"/>
-  <xacro:arg name="camera_far" default="3.0"/>
+  <xacro:arg name="camera_far" default="30.0"/>
+  <xacro:arg name="depth_camera_near" default="0.3"/>
+  <xacro:arg name="depth_camera_far" default="3.0"/>
   <xacro:arg name="camera_mass" default="0.030"/>
   <xacro:arg name="camera_size_x" default="0.0207"/>
@@ -128,4 +130,6 @@
   <xacro:property name="camera_near" value="$(arg camera_near)"/>
   <xacro:property name="camera_far" value="$(arg camera_far)"/>
+  <xacro:property name="depth_camera_near" value="$(arg depth_camera_near)"/>
+  <xacro:property name="depth_camera_far" value="$(arg depth_camera_far)"/>
   <xacro:property name="camera_width_m" value="$(arg camera_size_y)"/>
   <xacro:property name="camera_depth" value="$(arg camera_size_x)"/>

File: malbut_gazebo/urdf/gazebo_plugins.xacro (robot description, xacro)
@@ -135,4 +135,10 @@
               <far>${camera_far}</far>
             </clip>
+            <depth_camera>
+              <clip>
+                <near>${depth_camera_near}</near>
+                <far>${depth_camera_far}</far>
+              </clip>
+            </depth_camera>
           </camera>
         </sensor>

Commit message: fix(SWM25-46): ROSOrin 로봇 에셋 구성

File: malbut_description/urdf/rosorin_model.xacro (robot description, xacro)
@@ -13,4 +13,8 @@
   <xacro:arg name="wheel_radius" default="0.040"/>
   <xacro:arg name="wheel_width" default="0.03808"/>
+  <xacro:arg name="wheel_x_offset" default="0.0051465"/>
+  <xacro:arg name="wheel_y_offset" default="0.000074"/>
+  <xacro:arg name="front_wheel_z" default="0.017097"/>
+  <xacro:arg name="rear_wheel_z" default="0.016719"/>
   <xacro:arg name="wheel_joint_damping" default="0.02"/>
   <xacro:arg name="wheel_joint_friction" default="0.0"/>
@@ -22,19 +26,16 @@
   <xacro:arg name="drive_max_velocity" default="1.5"/>
   <xacro:arg name="odom_publish_frequency" default="50.0"/>
-  <xacro:arg name="base_mass" default="1.35"/>
+  <xacro:arg name="base_mass" default="2.163"/>
   <xacro:arg name="base_length" default="0.274"/>
-  <xacro:arg name="base_width" default="0.164"/>
-  <xacro:arg name="base_height" default="0.050"/>
-  <xacro:arg name="base_center_z" default="0.0"/>
-  <xacro:arg name="upper_body_mass" default="0.813"/>
-  <xacro:arg name="upper_body_length" default="0.170"/>
-  <xacro:arg name="upper_body_width" default="0.135"/>
-  <xacro:arg name="upper_body_height" default="0.085"/>
-  <xacro:arg name="upper_body_x" default="-0.012"/>
-  <xacro:arg name="upper_body_z" default="0.0825"/>
+  <xacro:arg name="base_width" default="0.163315"/>
+  <xacro:arg name="base_height" default="0.112562"/>
+  <xacro:arg name="base_footprint_z" default="0.028"/>
+  <xacro:arg name="base_com_x" default="-0.0073743"/>
+  <xacro:arg name="base_com_y" default="0.00027245"/>
+  <xacro:arg name="base_com_z" default="0.033869"/>
   <xacro:arg name="wheel_mass" default="0.10"/>
   <xacro:arg name="camera_x" default="0.057373"/>
   <xacro:arg name="camera_y" default="0.000079"/>
-  <xacro:arg name="camera_z" default="0.079864"/>
+  <xacro:arg name="camera_z" default="0.091864"/>
   <xacro:arg name="camera_roll" default="0.0"/>
   <xacro:arg name="camera_pitch" default="0.0"/>
@@ -54,5 +55,5 @@
   <xacro:arg name="lidar_x" default="0.011476"/>
   <xacro:arg name="lidar_y" default="0.000074"/>
-  <xacro:arg name="lidar_z" default="0.1086"/>
+  <xacro:arg name="lidar_z" default="0.13641"/>
   <xacro:arg name="lidar_roll" default="0.0"/>
   <xacro:arg name="lidar_pitch" default="0.0"/>
@@ -78,7 +79,7 @@
   <xacro:arg name="imu_size_y" default="0.020"/>
   <xacro:arg name="imu_size_z" default="0.005"/>
-  <xacro:arg name="microphone_x" default="-0.069"/>
-  <xacro:arg name="microphone_y" default="0.0"/>
-  <xacro:arg name="microphone_z" default="0.109"/>
+  <xacro:arg name="microphone_x" default="-0.068965"/>
+  <xacro:arg name="microphone_y" default="0.025075"/>
+  <xacro:arg name="microphone_z" default="0.10955"/>
   <xacro:arg name="microphone_mass" default="0.020"/>
   <xacro:arg name="microphone_diameter" default="0.104"/>
@@ -92,4 +93,8 @@
   <xacro:property name="wheel_radius" value="$(arg wheel_radius)"/>
   <xacro:property name="wheel_width" value="$(arg wheel_width)"/>
+  <xacro:property name="wheel_x_offset" value="$(arg wheel_x_offset)"/>
+  <xacro:property name="wheel_y_offset" value="$(arg wheel_y_offset)"/>
+  <xacro:property name="front_wheel_z" value="$(arg front_wheel_z)"/>
+  <xacro:property name="rear_wheel_z" value="$(arg rear_wheel_z)"/>
   <xacro:property name="wheel_joint_damping" value="$(arg wheel_joint_damping)"/>
   <xacro:property name="wheel_joint_friction" value="$(arg wheel_joint_friction)"/>
@@ -103,5 +108,4 @@
   <!-- Component masses are validated against total_mass by the main launch. -->
   <xacro:property name="base_mass" value="$(arg base_mass)"/>
-  <xacro:property name="upper_body_mass" value="$(arg upper_body_mass)"/>
   <xacro:property name="wheel_mass" value="$(arg wheel_mass)"/>
   <xacro:property name="camera_mass" value="$(arg camera_mass)"/>
@@ -112,10 +116,8 @@
   <xacro:property name="base_width" value="$(arg base_width)"/>
   <xacro:property name="base_height" value="$(arg base_height)"/>
-  <xacro:property name="base_center_z" value="$(arg base_center_z)"/>
-  <xacro:property name="upper_body_length" value="$(arg upper_body_length)"/>
-  <xacro:property name="upper_body_width" value="$(arg upper_body_width)"/>
-  <xacro:property name="upper_body_height" value="$(arg upper_body_height)"/>
-  <xacro:property name="upper_body_x" value="$(arg upper_body_x)"/>
-  <xacro:property name="upper_body_z" value="$(arg upper_body_z)"/>
+  <xacro:property name="base_footprint_z" value="$(arg base_footprint_z)"/>
+  <xacro:property name="base_com_x" value="$(arg base_com_x)"/>
+  <xacro:property name="base_com_y" value="$(arg base_com_y)"/>
+  <xacro:property name="base_com_z" value="$(arg base_com_z)"/>
   <xacro:property name="camera_x" value="$(arg camera_x)"/>
   <xacro:property name="camera_y" value="$(arg camera_y)"/>

File: malbut_gazebo/urdf/gazebo_plugins.xacro (robot description, xacro)
@@ -24,16 +24,4 @@
   </xacro:macro>
   <xacro:macro name="rosorin_gazebo">
-    <gazebo reference="base_link">
-      <material>Gazebo/Orange</material>
-    </gazebo>
-    <gazebo reference="upper_body_link">
-      <material>Gazebo/Grey</material>
-    </gazebo>
-    <gazebo reference="camera_link">
-      <material>Gazebo/DarkGrey</material>
-    </gazebo>
-    <gazebo reference="laser_frame">
-      <material>Gazebo/DarkGrey</material>
-    </gazebo>
     <!-- Same directional-friction approximation used by Fortress' mecanum demo. -->
     <xacro:mecanum_friction link="front_left_wheel_link" direction="1 -1 0"/>
@@ -82,10 +70,6 @@
       <gazebo reference="laser_frame">
         <sensor name="stl19p_d500" type="gpu_lidar">
-          <!--
-            The profile locates laser_frame at the D500 enclosure center.
-            Emit rays from the top scan plane so they do not intersect the
-            upper-body collision geometry directly below the sensor.
-          -->
-          <pose>0 0 ${lidar_height / 2.0} 0 0 0</pose>
+          <!-- Hiwonder defines laser_frame at the physical scan plane. -->
+          <pose>0 0 0 0 0 0</pose>
           <always_on>true</always_on>
           <update_rate>${lidar_rate}</update_rate>
